File: Atmega328P/AtMega328p-ethernet/AtMega328p-ethernet.kicad_sch (KiCad schematic)
At the start: 20 parts, among them J2 USB_C_Receptacle_USB2.0_16P, J3 RJ45_Abracon_ARJP11A-MASA-B-A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, SW1 SW_Push, U1 ATmega328P-A, U2 W5500, U3 MCP2200-I-SS, Y1 Crystal

Commit message: Continued work on ethernet
Parts:
- removed D3: LED, symbol Device:LED
- removed J2: USB_C_Receptacle_USB2.0_16P, symbol Connector:USB_C_Receptacle_USB2.0_16P
- removed J3: RJ45_Abracon_ARJP11A-MASA-B-A-EMU2, Connector_RJ:RJ45_Abracon_ARJP11A-MA_Horizontal, symbol Connector:RJ45_Abracon_ARJP11A-MASA-B-A-EMU2
- removed R4: 10k, symbol Device:R_Small
- removed U2: W5500, Package_QFP:LQFP-48_7x7mm_P0.5mm, symbol Interface_Ethernet:W5500
- removed U3: MCP2200-I-SS, Package_SO:SSOP-20_5.3x7.2mm_P0.65mm, symbol Interface_USB:MCP2200-I-SS
Connections:
- net SPI_ETH_SS renamed ETH_SPI_SS
Other:
- added sheet ETHERNET_MODULE (Ethernet.kicad_sch)
- added sheet USB_INTERFACE (Usb.kicad_sch)
- moved on the sheet: C1, C2, C3, C4, D1, D2, R1, R2, R3, R5, R6, SW1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
