File: Atmega328P/AtMega328p-ethernet/AtMega328p-ethernet.kicad_sch (KiCad schematic)
At the start: 28 parts, among them J10 Conn_02x03_Counter_Clockwise, J3 Conn_02x05_Odd_Even, J4 Conn_01x06_Socket, J5 Conn_01x06_Socket, J6 Conn_01x06_Socket, J7 Conn_01x06_Socket, J8 Conn_02x03_Counter_Clockwise, SW1 SW_Push, U1 ATmega328P-A, Y1 16MHz

Commit message: Most traces complete just GPIO left
Parts:
- added FB3: 100R@100MHz, Inductor_SMD:L_0603_1608Metric, symbol Device:FerriteBead_Small
Connections:
- net +5V: now also FB3.2
- net VBUS: now also FB3.1
Other:
- moved on the sheet: FB2
Changed lines of the file:
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@@
 	)
 	(junction
+		(at 290.83 88.9)
+		(diameter 0)
+		(color 0 0 0 0)
+	)
+	(junction
 		(at 377.19 38.1)
 		(diameter 0)
@@
 	)
 	(junction
+		(at 275.59 88.9)
+		(diameter 0)
+		(color 0 0 0 0)
+	)
+	(junction
 		(at 307.34 217.17)
 		(diameter 0)
@@
 	(wire
 		(pts
+			(xy 275.59 92.71) (xy 280.67 92.71)
+		)
+		(stroke
+			(width 0)
+			(type default)
+		)
+	)
+	(wire
+		(pts
 			(xy 62.23 71.12) (xy 59.69 71.12)
 		)
@@
 	(wire
 		(pts
-			(xy 280.67 88.9) (xy 271.78 88.9)
+			(xy 279.4 48.26) (xy 300.99 48.26)
 		)
 		(stroke
@@
 	(wire
 		(pts
-			(xy 279.4 48.26) (xy 300.99 48.26)
+			(xy 138.43 102.87) (xy 180.34 102.87)
 		)
 		(stroke
@@
 	(wire
 		(pts
-			(xy 138.43 102.87) (xy 180.34 102.87)
+			(xy 130.81 208.28) (xy 144.78 208.28)
 		)
 		(stroke
@@
 	(wire
 		(pts
-			(xy 130.81 208.28) (xy 144.78 208.28)
+			(xy 290.83 88.9) (xy 294.64 88.9)
 		)
 		(stroke
@@
 	(wire
 		(pts
+			(xy 290.83 92.71) (xy 285.75 92.71)
+		)
+		(stroke
+			(width 0)
+			(type default)
+		)
+	)
+	(wire
+		(pts
+			(xy 275.59 85.09) (xy 275.59 88.9)
+		)
+		(stroke
+			(width 0)
+			(type default)
+		)
+	)
+	(wire
+		(pts
 			(xy 138.43 64.77) (xy 154.94 64.77)
 		)
@@
 	(wire
 		(pts
-			(xy 285.75 88.9) (xy 294.64 88.9)
+			(xy 285.75 85.09) (xy 290.83 85.09)
 		)
 		(stroke
@@
 	(wire
 		(pts
+			(xy 275.59 88.9) (xy 275.59 92.71)
+		)
+		(stroke
+			(width 0)
+			(type default)
+		)
+	)
+	(wire
+		(pts
 			(xy 358.14 152.4) (xy 364.49 152.4)
 		)
@@
 	(wire
 		(pts
+			(xy 275.59 85.09) (xy 280.67 85.09)
+		)
+		(stroke
+			(width 0)
+			(type default)
+		)
+	)
+	(wire
+		(pts
 			(xy 142.24 200.66) (xy 142.24 213.36)
 		)
@@
 	(wire
 		(pts
+			(xy 275.59 88.9) (xy 271.78 88.9)
+		)
+		(stroke
+			(width 0)
+			(type default)
+		)
+	)
+	(wire
+		(pts
 			(xy 58.42 127) (xy 58.42 128.27)
 		)
@@
 	(wire
 		(pts
+			(xy 290.83 88.9) (xy 290.83 92.71)
+		)
+		(stroke
+			(width 0)
+			(type default)
+		)
+	)
+	(wire
+		(pts
 			(xy 307.34 217.17) (xy 307.34 212.09)
 		)
@@
 	(wire
 		(pts
+			(xy 290.83 85.09) (xy 290.83 88.9)
+		)
+		(stroke
+			(width 0)
+			(type default)
+		)
+	)
+	(wire
+		(pts
 			(xy 111.76 238.76) (xy 97.79 238.76)
 		)
@@
 	)
 	(symbol
+		(lib_id "Device:FerriteBead_Small")
+		(at 283.21 92.71 270)
+		(mirror x)
+		(unit 1)
+		(exclude_from_sim no)
+		(in_bom yes)
+		(on_board yes)
+		(dnp no)
+		(property "Reference" "FB3"
+			(at 283.21 95.758 90)
+			(effects
+				(font
+					(size 1.27 1.27)
+				)
+			)
+		)
+		(property "Value" "100R@100MHz"
+			(at 283.464 89.662 90)
+			(effects
+				(font
+					(size 1.27 1.27)
+				)
+			)
+		)
+		(property "Footprint" "Inductor_SMD:L_0603_1608Metric"
+			(at 283.21 94.488 90)
+			(effects
+				(font
+					(size 1.27 1.27)
+				)
+				(hide yes)
+			)
+		)
+		(property "Datasheet" "~"
+			(at 283.21 92.71 0)
+			(effects
+				(font
+					(size 1.27 1.27)
+				)
+				(hide yes)
+			)
+		)
+		(property "Description" "Ferrite bead, small symbol"
+			(at 283.21 92.71 0)
+			(effects
+				(font
+					(size 1.27 1.27)
+				)
+				(hide yes)
+			)
+		)
+		(property "LCSC" "C1015"
+			(at 283.21 92.71 0)
+			(effects
+				(font
+					(size 1.27 1.27)
+				)
+				(hide yes)
+			)
+		)
+		(pin "1"
+		)
+		(pin "2"
+		)
+		(instances
+			(project "AtMega328p-ethernet"
+				(path "/441f74dc-335f-4227-aefc-792ec34889a2"
+					(reference "FB3")
+					(unit 1)
+				)
+			)
+		)
+	)
+	(symbol
 		(lib_id "power:GND")
 		(at 320.04 220.98 0)
@@
 	(symbol
 		(lib_id "Device:FerriteBead_Small")
-		(at 283.21 88.9 270)
+		(at 283.21 85.09 270)
 		(mirror x)
 		(unit 1)
@@
 		(dnp no)
 		(property "Reference" "FB2"
-			(at 283.2481 82.55 90)
+			(at 283.2481 78.74 90)
 			(effects
 				(font
@@
 		)
 		(property "Value" "100R@100MHz"
-			(at 283.464 85.852 90)
+			(at 283.464 82.042 90)
 			(effects
 				(font
@@
 		)
 		(property "Footprint" "Inductor_SMD:L_0603_1608Metric"
-			(at 283.21 90.678 90)
+			(at 283.21 86.868 90)
 			(effects
 				(font
@@
 		)
 		(property "Datasheet" "~"
-			(at 283.21 88.9 0)
+			(at 283.21 85.09 0)
 			(effects
 				(font
@@
 		)
 		(property "Description" "Ferrite bead, small symbol"
-			(at 283.21 88.9 0)
+			(at 283.21 85.09 0)
 			(effects
 				(font
@@
 		)
 		(property "LCSC" "C1015"
-			(at 283.21 88.9 0)
+			(at 283.21 85.09 0)
 			(effects
 				(font

Commit message: Tracing complete ready for final check and silk screen.
Parts:
- added C23: 100nF, Capacitor_SMD:C_0603_1608Metric, symbol Device:C_Small
- R5, R6: now not fitted
Connections:
- net SCL is gone; now on net I2C_SCL: J3.6 (Pin_6)
- net SDA is gone; now on net I2C_SDA: J3.4 (Pin_4)
- net SPI_CLK is gone; now on net SPI_MOSI: J3.7 (Pin_7)
- net +3.3V: now also R5.2, R6.2
- net +5V: no longer R5.2, R6.2
- net GND: now also C23.2
- net PB0: now also J6.4 (Pin_4); no longer J6.3 (Pin_3)
- net PB1: now also J6.3 (Pin_3); no longer J6.4 (Pin_4)
- net PD2: now also J5.6 (Pin_6); no longer J5.3 (Pin_3)
- net PD3: now also J5.5 (Pin_5); no longer J5.4 (Pin_4)
- net PD4: now also J5.4 (Pin_4); no longer J5.5 (Pin_5)
- net PD5: now also J5.3 (Pin_3); no longer J5.6 (Pin_6)
- net PD6/LED1: now also D2.2 (A), J6.6 (Pin_6); no longer D1.2 (A), J6.5 (Pin_5)
- net PD7/LED2: now also D1.2 (A), J6.5 (Pin_5); no longer D2.2 (A), J6.6 (Pin_6)
- net SPI_MOSI: no longer J3.3 (Pin_3)
- net SPI_SCK: now also J3.3 (Pin_3)
- net at U1.20 (AREF): now also C23.1
- no-connect marks 2 -> 4
