File: ExpansionBoards/IOExpander16/IOExpander16.kicad_sch (KiCad schematic)
At the start: 20 parts, among them J1 Screw_Terminal_01x02, J10 Screw_Terminal_01x02, J11 Screw_Terminal_01x02, J12 Screw_Terminal_01x02, J13 Screw_Terminal_01x02, J14 Screw_Terminal_01x02, J15 Screw_Terminal_01x02, J16 Screw_Terminal_01x02, J2 Screw_Terminal_01x05, J3 Conn_02x05_Counter_Clockwise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

Commit message: IO expansion board layout compeleted ready for review.
Connections:
- net SCL: now also U1.22 (SCL); no longer U1.23 (SDA)
- net SDA: now also U1.23 (SDA); no longer U1.22 (SCL)
- net SPI_CLK: now also J3.3 (Pin_3); no longer J3.7 (Pin_7)
- net SPI_MOSI: now also J3.7 (Pin_7); no longer J3.3 (Pin_3)
